Commit message: fix d435 model error

File: home_bringup/urdf/home.urdf.xacro (robot description, xacro)
@@ -9,7 +9,10 @@
   <xacro:include filename="$(find kobuki_description)/urdf/kobuki.urdf.xacro" />
   <xacro:include filename="$(find home_bringup)/urdf/hexagons.urdf.xacro"/>
-  <xacro:include filename="$(find home_bringup)/urdf/d435.urdf.xacro"/>
+  <xacro:include filename="$(find realsense2_camera)/urdf/_d435.urdf.xacro"/>
   <kobuki/>
   <stack_hexagons parent="base_link"/>
   <sensor_kinect  parent="base_link"/>
+  <sensor_d435 parent="base_link">
+    <origin xyz="-0.05 0 1.38" rpy="0 0 0"/>
+  </sensor_d435>
 </robot>

File: home_bringup/urdf/turtlebot_common_library.urdf.xacro (robot description, xacro)
@@ -6,4 +6,4 @@
   <!-- General -->
   <xacro:include filename="$(find turtlebot_description)/urdf/common_properties.urdf.xacro"/>
-  <xacro:include filename="$(find turtlebot_description)/urdf/turtlebot_properties.urdf.xacro"/>
+  <!-- <xacro:include filename="$(find turtlebot_description)/urdf/turtlebot_properties.urdf.xacro"/> -->
 </robot>

File: home_bringup/urdf/turtlebot_properties.urdf.xacro (robot description, xacro)
@@ -19,7 +19,7 @@
      (currently in development and awaiting feedback)
    -->
-	<xacro:property name="cam_px" value="0" />
+	<xacro:property name="cam_px" value="-0.0500" />
 <!--	<xacro:property name="cam_py" value="-0.0125" /> Y varies for different configurations. get sets in sensors_urdf -->
-	<xacro:property name="cam_pz" value="1.2870" />
+	<xacro:property name="cam_pz" value="1.3800" />
 	<xacro:property name="cam_or" value="0" />
 	<xacro:property name="cam_op" value="0" />

Commit message: something won't be ideal

File: home_bringup/urdf/home.urdf.xacro (robot description, xacro)
@@ -14,5 +14,5 @@
   <sensor_kinect  parent="base_link"/>
   <sensor_d435 parent="base_link">
-    <origin xyz="-0.05 0 1.38" rpy="0 0 0"/>
+    <origin xyz="-0.05 0 1.15" rpy="0 0 0"/>
   </sensor_d435>
 </robot>
